File: Adrion_1/Adrion_1.kicad_sch (KiCad schematic)
At the start: 0 parts

Commit message: Desarrollo
Other:
- added sheet OVP (OVP.kicad_sch)
Changed lines of the file:
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@@
 	(paper "A4")
 	(sheet
-		(at 171.45 31.75)
+		(at 205.74 31.75)
 		(size 52.07 26.67)
 		(exclude_from_sim no)
@@
 		)
 		(property "Sheetname" "Supply"
-			(at 171.45 31.0384 0)
+			(at 205.74 31.0384 0)
 			(effects
 				(font
@@
 		)
 		(property "Sheetfile" "supply.kicad_sch"
-			(at 171.45 59.0046 0)
+			(at 205.74 59.0046 0)
 			(effects
 				(font
@@
 		)
 		(property "Field2" ""
-			(at 171.45 31.75 0)
+			(at 205.74 31.75 0)
 			(effects
 				(font
@@
 	)
 	(sheet
-		(at 99.06 31.75)
+		(at 29.21 72.39)
+		(size 54.61 27.94)
+		(exclude_from_sim no)
+		(in_bom yes)
+		(on_board yes)
+		(dnp no)
+		(fields_autoplaced yes)
+		(stroke
+			(width 0.1524)
+			(type solid)
+		)
+		(fill
+			(color 0 0 0 0.0000)
+		)
+		(property "Sheetname" "OVP"
+			(at 29.21 71.6784 0)
+			(effects
+				(font
+					(size 1.27 1.27)
+				)
+				(justify left bottom)
+			)
+		)
+		(property "Sheetfile" "OVP.kicad_sch"
+			(at 29.21 100.9146 0)
+			(effects
+				(font
+					(size 1.27 1.27)
+				)
+				(justify left top)
+			)
+		)
+		(instances
+			(project "Adrion_1"
+				(path "/ca8b9c62-24ed-451b-8ada-8e095e6c3e3b"
+					(page "5")
+				)
+			)
+		)
+	)
+	(sheet
+		(at 113.03 31.75)
 		(size 54.61 26.67)
 		(exclude_from_sim no)
@@
 		)
 		(property "Sheetname" "Control"
-			(at 99.06 31.0384 0)
+			(at 113.03 31.0384 0)
 			(effects
 				(font
@@
 		)
 		(property "Sheetfile" "untitled.kicad_sch"
-			(at 99.06 59.0046 0)
+			(at 113.03 59.0046 0)
 			(effects
 				(font

Commit message: Correcciones
Changed lines of the file:
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@@
 	)
 	(sheet
-		(at 113.03 31.75)
+		(at 116.84 31.75)
 		(size 54.61 26.67)
 		(exclude_from_sim no)
@@
 		)
 		(property "Sheetname" "Control"
-			(at 113.03 31.0384 0)
+			(at 116.84 31.0384 0)
 			(effects
 				(font
@@
 		)
 		(property "Sheetfile" "untitled.kicad_sch"
-			(at 113.03 59.0046 0)
+			(at 116.84 59.0046 0)
 			(effects
 				(font

Commit message: Correcion railes de tension papa
Other:
- removed sheet OVP
Changed lines of the file:
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@@
-	)
-	(sheet
-		(at 29.21 72.39)
-		(size 54.61 27.94)
-		(exclude_from_sim no)
-		(in_bom yes)
-		(on_board yes)
-		(dnp no)
-		(fields_autoplaced yes)
-		(stroke
-			(width 0.1524)
-			(type solid)
-		)
-		(fill
-			(color 0 0 0 0.0000)
-		)
-		(property "Sheetname" "OVP"
-			(at 29.21 71.6784 0)
-			(effects
-				(font
-					(size 1.27 1.27)
-				)
-				(justify left bottom)
-			)
-		)
-		(property "Sheetfile" "OVP.kicad_sch"
-			(at 29.21 100.9146 0)
-			(effects
-				(font
-					(size 1.27 1.27)
-				)
-				(justify left top)
-			)
-		)
-		(instances
-			(project "Adrion_1"
-				(path "/ca8b9c62-24ed-451b-8ada-8e095e6c3e3b"
-					(page "5")
-				)
-			)
-		)
 	)
 	(sheet
