File: Adrion_1/Power_Stage.kicad_sch (KiCad schematic)
At the start: 83 parts, among them IC4 CKSR_15-NP, J1 Screw_Terminal_01x02, J3 Conn_01x04, Q1 IPT034N15NM6ATMA1, Q2 IPT034N15NM6ATMA1, Q3 IPT034N15NM6ATMA1, Q5 IPT034N15NM6ATMA1, U1 UCC21521DW, U3 UCC21521DW

Commit message: Desarrollo
Parts:
- added C51, C59: 100n, symbol Device:C
- C14, C15, C16, C6, R23, R24, R25, R26: now not fitted
Connections:
- net GND: now also C51.1, C59.2
- net GNDPWR: now also R10.2, R9.2, U1.10 (OUTB)
- net VCC: no longer U1.8 (VCCI)
- net 1.65V: now reaches IC4.11 (VREF)
- net 1.65V: now also C59.1
- new net: C51.2, U1.8 (VCCI)
- no-connect marks 1 -> 0
Other:
- moved on the sheet: C39, C7, J3

Commit message: Correcciones
Parts:
- removed IC4: CKSR_15-NP, CKSR15NP, symbol CKSR_15-NP:CKSR_15-NP
- added U8: CKSR_6-NP, Sensor_Current:LEM_CKSR, symbol Sensor_Current:CKSR_6-NP
Connections:
- net +5V: now also U8.14 (U_{c})
- net 1.65V: now also U8.11 (U_{ref})
- net GND: now also U8.13 (GND)
- net at C14.1, C18.2, C19.2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: now also U8.2 (IN1), U8.3 (IN2), U8.4 (IN3), U8.5 (IN4)
- net at R27.1: now also U8.12 (U_{out})
- net at J1.1 (Pin_1): now also U8.6 (OUT4), U8.7 (OUT3), U8.8 (OUT2), U8.9 (OUT1)
- net ADC_IN renamed I_sense
Other:
- moved on the sheet: C17, R27

Commit message: Footprints
Parts:
- removed C36, C37, C42, C43, C44, C45, C46, C47, C48: 560uF, symbol Device:C_Polarized_US
- removed C38, C59: 100n, symbol Device:C
- removed C39, C41: 10u, symbol Device:C
- removed C49: 1000uF, symbol Device:C_Polarized_US
- removed D6: BAV70, Package_TO_SOT_SMD:SOT-23, symbol Diode:BAV70
- removed Q5: IPT034N15NM6ATMA1, IAUT150N10S5N035ATMA1, symbol IPT034N15NM6ATMA1:IPT034N15NM6ATMA1
- removed R26, R29, R32: R, symbol Device:R
- removed R27: 100, symbol Device:R
- removed R33: 10k, symbol Device:R
- added C27, C28, C29, C30, C31, C32, C33, C36, C37: B43547F2108M067, CAPPRD1000W190D3550H4200:CAPPRD1000W190D3550H4200, symbol B43547F2108M067:B43547F2108M067
- added C38: 1000u, CAPPRD1000W190D3550H4200:CAPPRD1000W190D3550H4200, symbol B43547F2108M067:B43547F2108M067
- added C39: 4.7 uF, MKP1F044706J00JSSD:MKP1F044706J00JSSD, symbol MKP1F044706J00JSSD:MKP1F044706J00JSSD
- added C41: MKP1F044706J00JSSD, MKP1F044706J00JSSD, symbol MKP1F044706J00JSSD:MKP1F044706J00JSSD
- added C44: 100n, Capacitor_SMD:C_0603_1608Metric_Pad1.08x0.95mm_HandSolder, symbol Device:C
- added C45, C46, C47: 1u, Capacitor_SMD:C_0805_2012Metric, symbol Device:C
- added C48: 100n, Capacitor_SMD:C_0603_1608Metric, symbol Device:C
- added D8: STPS20200CTN, TO255P460X1020X1905-3P:TO255P460X1020X1905-3P, symbol STPS20200CTN:STPS20200CTN
- added Q4: IPT034N15NM6ATMA1, IAUT150N10S5N035ATMA1:IAUT150N10S5N035ATMA1, symbol IPT034N15NM6ATMA1:IPT034N15NM6ATMA1
- added R16: 4.7, Resistor_SMD:R_0805_2012Metric_Pad1.20x1.40mm_HandSolder, symbol Device:R
- added R26, R27, R28: CRCW251215K0FKEG, RESC6332X70N:RESC6332X70N, symbol CRCW251215K0FKEG:CRCW251215K0FKEG
- added R5: 51, Resistor_SMD:R_0603_1608Metric_Pad0.98x0.95mm_HandSolder, symbol Device:R
- C1, C11, C2, C4, C51, C8: footprint (none) -> Capacitor_SMD:C_0603_1608Metric_Pad1.08x0.95mm_HandSolder; Field5 (none) -> 0603
- C10, C3: footprint (none) -> Capacitor_SMD:C_0603_1608Metric_Pad1.08x0.95mm_HandSolder
- C12, C13, C17, C18, C21, C23, C7: footprint (none) -> Capacitor_SMD:C_0603_1608Metric; Field5 (none) -> 0603
- C14, C15, C6: footprint (none) -> Capacitor_SMD:C_1206_3216Metric_Pad1.33x1.80mm_HandSolder; Field5 (none) -> 1206; now fitted
- C16: footprint (none) -> Capacitor_SMD:C_1206_3216Metric_Pad1.33x1.80mm_HandSolder; Field5 (none) -> 1206; Field6 (none) -> 1206; now fitted
- C19, C20, C22: footprint (none) -> Capacitor_SMD:C_1206_3216Metric; Field5 (none) -> 1206
- C24: value 100n -> 10u; footprint (none) -> Capacitor_SMD:C_1206_3216Metric; Field5 (none) -> 1206
- C25: value 10u -> 100n; footprint (none) -> Capacitor_SMD:C_0603_1608Metric; Field5 (none) -> 0603
- C40, C5: value 10u -> 1u; footprint (none) -> Capacitor_SMD:C_0805_2012Metric; Field5 (none) -> 0805
- C9: value 2.2nF -> 2.2n; footprint (none) -> Capacitor_SMD:C_0603_1608Metric_Pad1.08x0.95mm_HandSolder; Field5 (none) -> 0603
- D1, D2, D3, D4: footprint MICROSMP -> MSS1P4-M3_89A:MICROSMP
- PS2, PS3: footprint NCM3S1212MCR7 -> NCM3S1212MCR7:NCM3S1212MCR7
- Q1: footprint IAUT150N10S5N035ATMA1 -> IAUT150N10S5N035ATMA1:IAUT150N10S5N035ATMA1
- R1, R11, R15, R3, R8: footprint (none) -> Resistor_SMD:R_0603_1608Metric_Pad0.98x0.95mm_HandSolder; Field5 (none) -> 0603
- R10, R17, R18, R6, R7, R9: footprint (none) -> Resistor_SMD:R_0805_2012Metric_Pad1.20x1.40mm_HandSolder; Field5 (none) -> 0805
- R12: value 51 -> 10k; footprint (none) -> Resistor_SMD:R_0603_1608Metric_Pad0.98x0.95mm_HandSolder; Field5 (none) -> 0603
- R13: value 51 -> 25k; footprint (none) -> Resistor_SMD:R_0603_1608Metric_Pad0.98x0.95mm_HandSolder; Field5 (none) -> 0603
- R14: value 25k -> 4.7; footprint (none) -> Resistor_SMD:R_0805_2012Metric_Pad1.20x1.40mm_HandSolder; Field5 (none) -> 0805
- R19, R20: value 4.7 -> 10k; footprint (none) -> Resistor_SMD:R_0603_1608Metric_Pad0.98x0.95mm_HandSolder; Field5 (none) -> 0603
- R2: footprint (none) -> Resistor_SMD:R_0603_1608Metric_Pad0.98x0.95mm_HandSolder
- R21, R22: value 10k -> R; footprint (none) -> Resistor_SMD:R_1206_3216Metric_Pad1.30x1.75mm_HandSolder; Field5 (none) -> 1206
- R23, R24: footprint (none) -> Resistor_SMD:R_1206_3216Metric_Pad1.30x1.75mm_HandSolder; Field5 (none) -> 1206; now fitted
- R25: value R -> 100; footprint (none) -> Resistor_SMD:R_0603_1608Metric_Pad0.98x0.95mm_HandSolder; Field5 (none) -> 0603; now fitted
- R4: value 10k -> 51; footprint (none) -> Resistor_SMD:R_0603_1608Metric_Pad0.98x0.95mm_HandSolder
- U1, U3: footprint UCC21521DW:SOIC127P1030X265-16N -> SOIC127P1030X265-16N:SOIC127P1030X265-16N
Connections:
- net 1.65V: now also C25.1
- net EN_GLOBAL: now also R12.1; no longer R4.1
- net GND: now also C18.2, C21.2, R12.2, R13.1, C44.1; no longer C23.2, R14.1, R4.2
- net GNDPWR: now also Q1.12 (S_8), Q2.12 (S_8), R23.2, C27.2, C28.2, C29.2, C30.2, C31.2, C32.2, C33.2, C36.2, C37.2, C38.2, C39.2, C41.2, C45.1, C46.1, C47.2, C48.2, R26.1, R27.1, R28.1; no longer C12.2, C7.2, R10.2, R19.2, R22.2, R9.2, U1.10 (OUTB), U3.10 (OUTB)
- net HV: now also C27.1, C28.1, C29.1, C30.1, C31.1, C32.1, C33.1, C36.1, C37.1, C38.1, C39.1, C41.1, D8.2, Q4.10 (D_2), Q4.11 (D_3), Q4.9 (D_1), R26.2, R27.2, R28.2; no longer Q3.12 (S_8)
- net I_sense: now also R25.2
- net PWM_BH: now also R4.1; no longer R12.1
- net PWM_BL: now also R5.1; no longer R13.1
- net VCC: no longer U3.8 (VCCI)
- net VDD: now also C18.1, C21.1, C45.2, C46.2, C47.1, C48.1; no longer C12.1, C23.1, C25.1, C7.1
- net at C14.1, C19.2, C5.2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: now also C12.1, C7.2, R21.2, Q4.12 (S_8), Q4.2 (S_1), Q4.3 (S_2), Q4.4 (S_3), Q4.5 (S_4), Q4.6 (S_5), Q4.7 (S_6), Q4.8 (S_7); no longer C18.2, Q1.12 (S_8), R23.2
- net at C15.2: now also R22.1; no longer R25.1
- net at C8.2, U3.1 (INA): now also R4.2; no longer R12.2
- net at C13.2, C16.1, C20.2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: now also C23.2, Q3.12 (S_8), R19.2, R22.2; no longer C21.2, Q2.12 (S_8), R21.2, R25.2
- net at R17.2, R18.2: now also U3.10 (OUTB); no longer U3.15 (OUTA)
- net at C13.1, C20.1, C40.1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: now also C23.1; no longer C21.1
- net at C10.2, U3.2 (INB): now also R5.2; no longer R13.2
- net at C9.1, U3.6 (DT): now also R13.2; no longer R14.2
- net at D1.2, R6.1, R8.1: now also Q4.1 (G)
- net at C19.1, C5.1, PS2.3 (+VOUT)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: now also C12.2, C7.1; no longer C18.1
- net at U8.12 (U_{out}): now also R25.1
- net at D4.2, Q2.1 (G), R20.1: now also R18.1; no longer R22.1
- net at D4.1: now also R17.1; no longer R19.1
- net at D3.2, Q3.1 (G): now also R19.1, R16.1; no longer R18.1, R21.1
- net at R23.1: now also C16.2; no longer C6.2
- net at D3.1: now also R14.1; no longer R17.1
- net at J3.4 (Pin_4): now also D8.1, D8.3
- new net: R14.2, R16.2, U3.15 (OUTA)
- new net: C44.2, U3.8 (VCCI)
- new net: R10.2, R9.2, U1.10 (OUTB)
- new net: C6.2, R21.1
Other:
- moved on the sheet: C13, C40, D2, J3, Q3, R1

Commit message: Footprints
Parts:
- added C50, C54, C55, C58: 10u, Capacitor_SMD:C_1206_3216Metric, symbol Device:C
- added C52, C53, C56, C57: 100n, Capacitor_SMD:C_0603_1608Metric, symbol Device:C
- added PS1, PS4: NCM3S1212MC-R7, NCM3S1212MCR7:NCM3S1212MCR7, symbol NCM3S1212MC-R7:NCM3S1212MC-R7
Connections:
- net GND: now also C53.2, C54.2, C57.2, C58.2, PS1.1 (-VIN), PS4.1 (-VIN)
- net GNDPWR: now also C50.2, C52.2, C55.2, C56.2, PS1.4 (-VOUT), PS4.4 (-VOUT)
- net VDD: now also C53.1, C54.1, C57.1, C58.1, PS1.2 (+VIN), PS4.2 (+VIN); no longer C45.2, C46.2, C47.1, C48.1, U1.11 (VDDB), U3.11 (VDDB)
- new net: C45.2, C46.2, C50.1, C52.1, PS1.3 (+VOUT), U3.11 (VDDB)
- new net: C47.1, C48.1, C55.1, C56.1, PS4.3 (+VOUT), U1.11 (VDDB)
Other:
- moved on the sheet: C1, C12, C14, C16, C17, C18, C19, C2, C22, C25, C3, C39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

Commit message: meduelelacabeza
Parts:
- removed J1: Screw_Terminal_01x02, symbol Connector:Screw_Terminal_01x02
- removed J3: Conn_01x04, symbol Connector_Generic:Conn_01x04
- added J1, J2: 1705469, 1705469, symbol 1705469:1705469
Connections:
- net GNDPWR: now also J2.1
- net VCC: no longer C4.2, U1.3 (VCCI-1)
- net at C13.2, C16.1, C20.2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: now also J1.2
- net at D8.1, D8.3: now also J2.2
- net at U8.6 (OUT4), U8.7 (OUT3), U8.8 (OUT2)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: now also J1.1
- net VDD renamed 12V
- new net 3.3V: C4.2, U1.3 (VCCI-1)
