File: Adrion_1/supply.kicad_sch (KiCad schematic)
At the start: 17 parts, among them IC2 L6986H, IC3 TPS7A2030PDBVR

Commit message: Modificaciones
Other:
- moved on the sheet: C26, C27, C28, C29, C30, C31, C32, C33, C34, C35, IC2, IC3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

Commit message: Desarrollo
Parts:
- added C50: 1u, symbol Device:C
- added C56, C57, C58: 100n, symbol Device:C
- added R40, R41: 10k, symbol Device:R
- added R42: 10, symbol Device:R
- added U7: TLV9001IDCKR, TLV9001IDCKR:SOT65P210X110-5N, symbol TLV9001IDCKR:TLV9001IDCKR
Connections:
- net 3.3V: now also C57.1, R41.1, U7.5 (V+)
- net GND: now also C50.2, C56.2, C57.2, C58.2, R40.2
- new net: C58.1, U7.2 (V-)
- new net: C50.1, C56.1, R40.1, R41.2, U7.1 (IN+)
- new net: R42.1, U7.3 (IN-), U7.4 (OUT)
- new net 1.65V: R42.2

Commit message: Correcciones
Other:
- moved on the sheet: C26, C27, C28, C29, C30, C31, C32, C33, C34, C35, C50, C56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

Commit message: Correcion railes de tension papa
Parts:
- removed C27: 330p, symbol Device:C
- removed C28: 2.2p, symbol Device:C
- removed C29: 10n, symbol Device:C
- removed C30: 68n, symbol Device:C
- removed C31: 470n, symbol Device:C
- removed C32, C50: 1u, symbol Device:C
- removed C33: 10u, symbol Device:C
- removed C56, C57, C58: 100n, symbol Device:C
- removed IC2: L6986H, SOP65P640X120-17N, symbol L6986H:L6986H
- removed L1: 10u, symbol Device:L
- removed R16: 240k, symbol Device:R
- removed R30: 82k, symbol Device:R
- removed R31: 75k, symbol Device:R
- removed R40, R41: 10k, symbol Device:R
- removed R42: 10, symbol Device:R
- removed R5: R, symbol Device:R
- removed U7: TLV9001IDCKR, TLV9001IDCKR:SOT65P210X110-5N, symbol TLV9001IDCKR:TLV9001IDCKR
- added C52, C54: 10u, symbol Device:C
- added C53: 100n, symbol Device:C
- added D5: D22V0H1U2LP-7B, D22V0H1U2LP7B, symbol D22V0H1U2LP-7B:D22V0H1U2LP-7B
- added D7: SS3P4-M3_85A, SS3P4M385A, symbol SS3P4-M3_85A:SS3P4-M3_85A
- added G1: TLF80511TF_V50, TLF80511TF_V50:INF-PG-TO252-3-11_N, symbol TLF80511TF_V50:TLF80511TF_V50
- added IC1: REF1933AIDDCR, SOT95P280X110-5N, symbol REF1933AIDDCR:REF1933AIDDCR
- C26: value C -> 1u
Connections:
- net 1.65V: now also IC1.1 (VBIAS)
- net 5V: now also C54.1, G1.3 (Q), IC1.3 (EN), IC1.4 (VIN)
- net GND: now also C52.2, C53.2, C54.2, D5.2 (A), G1.2 (GND), IC1.2 (GND)
- net VDD: now also D7.2 (A)
- new net: C52.1, C53.1, D5.1 (K), D7.1 (K), G1.1 (I)
- new net 3V3: IC1.5 (VREF)
Other:
- moved on the sheet: C34, C35, IC3

Commit message: Footprints
Parts:
- removed IC3: TPS7A2030PDBVR, SOT95P280X145-5N, symbol TPS7A2030PDBVR:TPS7A2030PDBVR
- added U4: TPS7A2033PDBVR, TPS7A2033PDBVR:SOT95P280X145-5N, symbol TPS7A2033PDBVR:TPS7A2033PDBVR
Connections:
- net 3.3V: now also U4.5 (OUT)
- net 5V: now also U4.1 (IN)
- net ENABLE_LDO: now also U4.3 (EN)
- net GND: now also U4.2 (GND)
Other:
- moved on the sheet: C34

Commit message: Footprints
Parts:
- removed C52, C54: 10u, symbol Device:C
- removed C53: 100n, symbol Device:C
- added C42, C43: 10u, Capacitor_SMD:C_1206_3216Metric, symbol Device:C
- added C49: 100n, Capacitor_SMD:C_0603_1608Metric, symbol Device:C
- C26, C34, C35: footprint (none) -> Capacitor_SMD:C_0805_2012Metric; Field5 (none) -> 0805
- D5: footprint D22V0H1U2LP7B -> D22V0H1U2LP7B:D22V0H1U2LP7B
- D7: footprint SS3P4M385A -> SS3P4M385A:SS3P4M385A
- G1: footprint TLF80511TF_V50:INF-PG-TO252-3-11_N -> INF-PG-TO252-3-11_N:INF-PG-TO252-3-11_N
- IC1: footprint SOT95P280X110-5N -> SOT95P280X110-5N:SOT95P280X110-5N
- U4: footprint TPS7A2033PDBVR:SOT95P280X145-5N -> SOT95P280X145-5N:SOT95P280X145-5N
Connections:
- net ENABLE_LDO is gone; now on net 5V: U4.3 (EN)
- net 3.3V: now also C34.2; no longer C34.1
- net 5V: now also C43.1
- net GND: now also C34.1, C42.2, C43.2, C49.1; no longer C34.2
- net at D5.1 (K), D7.1 (K), G1.1 (I): now also C42.1, C49.2

Commit message: meduelelacabeza
Parts:
- added J4: 1729128, 1729128:PHOENIX_1729128, symbol 1729128:1729128
Connections:
- net GND: now also J4.1
- net VDD renamed 12V
- net 12V: now also J4.2

Commit message: Mamita he empezado el layout. Vaya show
Parts:
- removed J4: 1729128, 1729128:PHOENIX_1729128, symbol 1729128:1729128
- added J3: 1729128, 1729128_2.0:1729128, symbol 1729128_2.0:1729128
Connections:
- net 12V: now also J3.2
- net GND: now also J3.1
- net 3V3: no longer names the net of IC1.5 (VREF)
- no-connect marks 0 -> 1
