File: Adrion_1/Adrion_1.kicad_pcb (KiCad board)
At the start: 4 copper layers, 193.4 x 230.1 mm, 112 parts, among them IC1 REF1933AIDDCR, IC2 UCC21521DW, IC3 UCC21521DW, J1 1705469, J2 1705469, J3 1729128, J6 M20-7821546, J7 M20-7821546, Q1 IPP111N15N3GXKSA1, Q2 IPP111N15N3GXKSA1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

Commit message: Layout
Parts:
- removed C36: B43547F2108M067, CAPPRD1000W190D3550H4200:CAPPRD1000W190D3550H4200
- added C30: B43547F2108M067, CAPPRD1000W190D3550H4200:CAPPRD1000W190D3550H4200, F.Cu at (155.0, 172.0)
- moved R28 196.9 mm to (161.0, 33.0), turned to -90 degrees
- moved R26 194.0 mm to (155.0, 33.0), turned to -90 degrees
- moved R27 192.3 mm to (149.0, 33.0), turned to -90 degrees
- moved C39 184.8 mm to (57.8, 219.0), turned to 180 degrees
- moved C41 158.3 mm to (58.8, 194.0)
- moved J2 134.2 mm to (156.5, 233.3), turned to 0 degrees
- moved D8 103.6 mm to (156.4, 215.3), turned to 0 degrees
- moved R12 92.2 mm to (29.0, 44.0)
- moved C20 43.0 mm to (72.0, 129.0)
- moved C40 39.6 mm to (32.0, 124.8)
- moved C53 37.3 mm to (34.0, 158.0)
- moved C58 35.8 mm to (35.0, 130.0)
- moved C23 35.4 mm to (67.0, 129.8), turned to 90 degrees
- moved R19 33.8 mm to (68.0, 141.0), turned to 180 degrees
- moved C52 30.7 mm to (65.5, 165.5)
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Routing:
- net Net-(D8-Pad1): track 31.8 -> 0.00 mm
- net Net-(IC3-VDDB): track 33.3 -> 8.81 mm
- net Net-(IC2-VSSA): track 0.00 -> 16.6 mm, vias 0 -> 2
- net Net-(IC3-VSSA): track 25.3 -> 13.1 mm, vias 2 -> 1
- net Net-(IC2-VDDB): track 0.00 -> 10.8 mm
- net Net-(Q1-G): track 9.77 -> 0.00 mm
- net Net-(IC2-OUTB): track 0.00 -> 5.98 mm
- net HV: track 5.65 -> 0.00 mm
- net Net-(IC2-VDDA): track 0.00 -> 5.27 mm
- net GNDPWR: track 15.8 -> 10.7 mm, vias 126 -> 1
- net Net-(IC2-OUTA): track 0.00 -> 4.62 mm
- net Net-(C14-Pad2): track 2.89 -> 0.00 mm
- net Net-(D2-Pad1): track 0.00 -> 2.56 mm
- net Net-(C6-Pad2): track 2.39 -> 0.00 mm
- net Net-(D3-Pad1): track 0.00 -> 2.00 mm
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- added copper zone on In2.Cu, net HV
- added copper zone on F.Cu, net Net-(D8-Pad1)
- added copper zone on F.Cu, net Net-(Q1-G)
- added copper zone on F.Cu, net Net-(Q2-G)
- added copper zone on F.Cu, net Net-(Q3-G)
- removed copper zone on F.Cu, net Net-(IC3-VSSA)
Other:
- board size 193.4 x 230.1 mm -> 193 x 231.1 mm

Commit message: Routing, Placement, Datasheets actualizado
Parts:
- removed C41: MKP1F044706J00JSSD, MKP1F044706J00JSSD:MKP1F044706J00JSSD
- removed G1: TLF80511TF_V50, INF-PG-TO252-3-11_N:INF-PG-TO252-3-11_N
- removed the R12 at (51.2, 148.2)
- added C36: C5750X6S2W225K250KA, C5750_Commercial:C5750_Commercial, B.Cu at (136.3, 81.9)
- added C37: C5750X6S2W225K250KA, C5750_Commercial:C5750_Commercial, B.Cu at (144.8, 81.9)
- added C59: C5750X6S2W225K250KA, C5750_Commercial:C5750_Commercial, B.Cu at (137.0, 51.8)
- added IC4: TLF80511TFV50ATMA1, IDD09E60:IDD09E60, F.Cu at (34.3, 51.7)
- C12, C18, C19, C20, C22, C23, C40, C44, C45, C52, C53, C54, C55, C56, C57, C58, PS1, PS2, PS3, PS4: moved to B.Cu
- C39: value 4.7 uF -> C5750X6S2W225K250KA; footprint MKP1F044706J00JSSD:MKP1F044706J00JSSD -> C5750_Commercial:C5750_Commercial; moved to B.Cu
- moved C39 188.6 mm to (145.0, 51.8), turned to 90 degrees
- moved U3 140.2 mm to (54.1, 163.4)
- moved R12 90.5 mm to (97.2, 103.5), turned to -90 degrees
- moved C44 88.9 mm to (83.5, 92.7)
- moved PS1 86.5 mm to (100.0, 94.2)
- moved J2 78.5 mm to (97.7, 181.2)
- moved D8 77.8 mm to (97.9, 164.0)
- moved R4 74.1 mm to (94.2, 97.0), turned to 0 degrees
- moved J1 72.9 mm to (148.0, 21.8), turned to 180 degrees
- moved C58 72.0 mm to (81.8, 75.2), turned to -90 degrees
- moved C8 71.6 mm to (98.8, 99.8), turned to 90 degrees
- moved R5 70.2 mm to (94.3, 98.8), turned to 0 degrees
- moved U5 69.8 mm to (139.0, 36.8), turned to 0 degrees
- moved C23 67.1 mm to (119.2, 87.8), turned to -90 degrees
- moved D2 66.2 mm to (118.5, 97.8)
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Connections:
- C39 pad 1: HV -> GNDPWR
- C39 pad 2: GNDPWR -> HV
Routing:
- net 12V: track 0.00 -> 229.3 mm, vias 0 -> 2
- net 5V: track 0.00 -> 140.4 mm
- net EN_B: track 0.00 -> 105.3 mm, vias 0 -> 2
- net Net-(IC2-VSSA): track 16.6 -> 121.3 mm, vias 2 -> 0
- net PWM_BH: track 0.00 -> 95.9 mm
- net PWM_BL: track 0.00 -> 94.9 mm, vias 0 -> 2
- net GND: track 0.46 -> 88.5 mm, vias 0 -> 17
- net PWM_AL: track 0.00 -> 69.5 mm, vias 0 -> 2
- net I_Sense: track 0.00 -> 53.1 mm
- net Net-(IC3-VSSA): track 13.1 -> 57.6 mm, vias 1 -> 0
- net PWM_AH: track 0.00 -> 36.0 mm
- net Net-(D5-K): track 0.43 -> 33.1 mm
- net 1.65V: track 0.00 -> 28.6 mm, vias 0 -> 2
- net Net-(U5-VOUT): track 0.00 -> 22.2 mm
- net Net-(U5-OUT_1): track 0.00 -> 16.5 mm
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- added copper zone on In1.Cu, net GND
- added copper zone on B.Cu, net GNDPWR
- added copper zone on F.Cu, net Net-(IC2-VSSA)
- added copper zone on F.Cu, net Net-(IC3-VSSA)
Other:
- board size 193 x 231.1 mm -> 215.2 x 179.8 mm

Commit message: arrreglos, venitilador y disipadores primera version
Parts:
- added HS1: 577202B04000G, HSINK_577202B04000G:HSINK_577202B04000G, F.Cu at (147.5, 58.9)
- added HS2: 577202B04000G, HSINK_577202B04000G:HSINK_577202B04000G, F.Cu at (147.6, 73.3)
- added HS3: 577202B04000G, HSINK_577202B04000G:HSINK_577202B04000G, F.Cu at (147.7, 89.8)
- added HS4: 577202B04000G, HSINK_577202B04000G:HSINK_577202B04000G, F.Cu at (147.7, 104.1)
- added U1: ~, 1705469:Untitled, F.Cu at (160.7, 178.8)
- moved U3 140.4 mm to (54.8, 23.0)
- moved C13 42.9 mm to (100.5, 107.0)
- moved C17 33.3 mm to (125.5, 42.0)
- moved C55 25.1 mm to (116.2, 73.5)
- moved C56 18.2 mm to (114.2, 74.0)
- moved R12 9.10 mm to (88.3, 105.3)
- moved C19 8.09 mm to (116.8, 55.5), turned to -90 degrees
- moved C45 7.28 mm to (116.2, 117.0)
- moved C23 7.23 mm to (114.0, 92.7), turned to 90 degrees
- moved C1 7.05 mm to (94.0, 63.5), turned to -90 degrees
- moved C12 6.99 mm to (114.2, 55.7), turned to 90 degrees
- moved C52 6.92 mm to (114.2, 117.0)
- moved C8 5.77 mm to (100.5, 94.2), turned to -90 degrees
- moved C3 5.14 mm to (100.0, 54.5), turned to 0 degrees
- moved C10 4.03 mm to (100.5, 97.8), turned to -90 degrees
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Routing:
- net 3.3V: track 3.85 -> 191.3 mm, vias 0 -> 6
- net EN_A: track 0.00 -> 70.1 mm, vias 0 -> 2
- net GNDPWR: track 15.9 -> 80.4 mm, vias 0 -> 3
- net HV: track 0.00 -> 41.3 mm, vias 0 -> 3
- net 5V: track 140.4 -> 160.6 mm
- net GND: track 88.5 -> 106.0 mm, vias 17 -> 26
- net Net-(IC3-VDDB): track 8.81 -> 23.9 mm, vias 0 -> 1
- net Net-(IC2-VDDB): track 10.8 -> 25.7 mm, vias 0 -> 1
- net Net-(IC3-DT): track 0.00 -> 10.2 mm
- net Net-(IC3-VDDA): track 4.73 -> 13.9 mm
- net Net-(IC3-INA): track 0.00 -> 7.88 mm
- net Net-(IC2-VDDA): track 5.27 -> 12.8 mm
- net Net-(IC3-INB): track 0.00 -> 7.56 mm
- net Net-(IC2-INB): track 1.81 -> 7.57 mm
- net PWM_AL: track 69.5 -> 74.5 mm
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
Commit message: FirstPrototype
First Prototype sent
Parts:
- removed C33: B43547F2108M067, CAPPRD1000W190D3550H4200:CAPPRD1000W190D3550H4200
- removed C38: 1000u, CAPPRD1000W190D3550H4200:CAPPRD1000W190D3550H4200
- removed HS1, HS2, HS3, HS4: 577202B04000G, HSINK_577202B04000G:HSINK_577202B04000G
- removed J6, J7: M20-7821546, HARWIN_M20-7821546:HARWIN_M20-7821546
- removed R28: CRCW251215K0FKEG, RESC6332X70N:RESC6332X70N
- removed U1: ~, 1705469:Untitled
- removed U3: NUCLEO-G431KB, MODULE_NUCLEO-G431KB:MODULE_NUCLEO-G431KB
- added C41: LGU2D102MELA, LGU2D102MELA:LGU2D102MELA, F.Cu at (180.0, 111.0)
- added C60: LGU2D102MELA, LGU2D102MELA:LGU2D102MELA, B.Cu at (194.8, 148.3)
- added J4: 7462810, 7462810:7462810, F.Cu at (137.3, 156.0)
- added J5: 7462810, 7462810:7462810, F.Cu at (155.0, 85.0)
- added J8: 6-534237-3, TE_6-534237-3:TE_6-534237-3, F.Cu at (86.2, 89.7)
- added J9: 6-534237-3, TE_6-534237-3:TE_6-534237-3, F.Cu at (101.3, 89.7)
- added R29: CRGP2512F15K, RESC6332X65N:RESC6332X65N, F.Cu at (207.8, 81.7)
- added REF**: MountingHole_3.2mm_M3_DIN965_Pad, MountingHole:MountingHole_3.2mm_M3_DIN965_Pad, F.Cu at (86.3, 155.1)
- added REF**: MountingHole_3.2mm_M3_DIN965_Pad, MountingHole:MountingHole_3.2mm_M3_DIN965_Pad, F.Cu at (210.1, 51.7)
- added REF**: MountingHole_3.2mm_M3_DIN965_Pad, MountingHole:MountingHole_3.2mm_M3_DIN965_Pad, F.Cu at (210.2, 155.8)
- added REF**: MountingHole_3.2mm_M3_DIN965_Pad, MountingHole:MountingHole_3.2mm_M3_DIN965_Pad, F.Cu at (86.2, 52.0)
- added REF**: MountingHole_3.2mm_M3_Pad, MountingHole:MountingHole_3.2mm_M3_Pad, F.Cu at (86.2, 52.0)
- added REF**: MountingHole_3.2mm_M3_Pad, MountingHole:MountingHole_3.2mm_M3_Pad, F.Cu at (210.1, 51.7)
- added REF**: MountingHole_3.2mm_M3_Pad, MountingHole:MountingHole_3.2mm_M3_Pad, F.Cu at (86.2, 155.1)
- added REF**: MountingHole_3.2mm_M3_Pad, MountingHole:MountingHole_3.2mm_M3_Pad, F.Cu at (210.3, 155.9)
- added TP1: TestPoint, TestPoint:TestPoint_Pad_D1.0mm, F.Cu at (103.0, 51.5)
- added TP2: TestPoint, TestPoint:TestPoint_Pad_D1.0mm, F.Cu at (99.1, 57.9)
- added TP3: TestPoint, TestPoint:TestPoint_Pad_D1.0mm, F.Cu at (87.5, 131.9)
- added TP4: TestPoint, TestPoint:TestPoint_Pad_D1.0mm, F.Cu at (111.2, 91.3)
- added TP5: TestPoint, TestPoint:TestPoint_Pad_D1.0mm, F.Cu at (118.7, 93.8)
- added TP6: TestPoint, TestPoint:TestPoint_Pad_D1.0mm, F.Cu at (103.0, 131.5)
- C12, C18, C19, C20, C22, C23, C40, C44, C45, C52, C53, C54, C55, C56, C57, C58: moved to F.Cu
- C14, C46, C50, C6, R21, R22, R23, R24: moved to B.Cu
- C27, C29, C31: value B43547F2108M067 -> LGU2D102MELA; footprint CAPPRD1000W190D3550H4200:CAPPRD1000W190D3550H4200 -> LGU2D102MELA:LGU2D102MELA
- C28, C30, C32: value B43547F2108M067 -> LGU2D102MELA; footprint CAPPRD1000W190D3550H4200:CAPPRD1000W190D3550H4200 -> LGU2D102MELA:LGU2D102MELA; moved to B.Cu
- D8: value STPS20200CTN -> SDT40A120CT; footprint TO255P460X1020X1905-3P:TO255P460X1020X1905-3P -> TO254P1066X482X2286-3:TO254P1066X482X2286-3
- J1, J2: value 1705469 -> 7462810; footprint 1705469:1705469 -> 7462810:7462810
- R26, R27: value CRCW251215K0FKEG -> CRGP2512F15K; footprint RESC6332X70N:RESC6332X70N -> RESC6332X65N:RESC6332X65N
- moved IC4 107.6 mm to (97.1, 139.1), turned to 90 degrees
- moved C43 100.8 mm to (96.8, 131.7), turned to 0 degrees
- moved C49 100.2 mm to (102.5, 134.7), turned to -90 degrees
- moved C29 93.2 mm to (180.0, 138.4), turned to -90 degrees
- moved C30 90.9 mm to (194.9, 66.6), turned to 90 degrees
- moved C42 88.1 mm to (102.2, 126.3), turned to -90 degrees
- moved D5 81.6 mm to (105.9, 126.2)
- moved D7 80.0 mm to (97.1, 126.3), turned to 180 degrees
- moved C39 77.9 mm to (138.4, 129.4), turned to 0 degrees
- moved C32 77.9 mm to (194.8, 121.0), turned to 90 degrees
- moved J1 75.5 mm to (162.9, 95.6), turned to 0 degrees
- moved C27 72.4 mm to (180.0, 83.7), turned to -90 degrees
- moved C31 71.5 mm to (180.0, 56.4), turned to -90 degrees
- moved R3 71.2 mm to (119.3, 120.3)
- moved R25 71.2 mm to (117.7, 97.2), turned to 180 degrees
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Connections:
- J1 pad 2: Net-(IC2-VSSA) -> Net-(U5-OUT_1)
- J2 pad 2: Net-(D8-Pad1) -> GNDPWR
- R26 pad 1: GNDPWR -> HV
- R26 pad 2: HV -> GNDPWR
- R27 pad 1: GNDPWR -> HV
- R27 pad 2: HV -> GNDPWR
Routing:
- net 12V: track 229.3 -> 34.6 mm, vias 2 -> 4
- net Net-(IC2-VSSA): track 121.8 -> 45.1 mm
- net PWM_BH: track 95.5 -> 34.2 mm, vias 0 -> 1
- net 3.3V: track 191.3 -> 131.3 mm, vias 6 -> 5
- net EN_B: track 106.3 -> 51.7 mm
- net PWM_BL: track 94.9 -> 49.5 mm, vias 2 -> 1
- net GNDPWR: track 80.4 -> 123.4 mm, vias 3 -> 6
- net I_Sense: track 53.1 -> 15.5 mm
- net Net-(IC3-VSSA): track 61.9 -> 39.2 mm
- net 1.65V: track 29.6 -> 10.6 mm, vias 2 -> 0
- net 5V: track 160.6 -> 178.4 mm, vias 0 -> 4
- net PWM_AH: track 36.0 -> 52.9 mm, vias 0 -> 1
- net Net-(U5-OUT_1): track 16.5 -> 0.00 mm
- net Net-(U5-VOUT): track 22.2 -> 7.56 mm
- net GND: track 106.0 -> 93.7 mm, vias 26 -> 51
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- added copper zone on In2.Cu, net 12V
- added copper zone on B.Cu, net GND
- added copper zone on F.Cu, net GND
- added copper zone on F.Cu, net Net-(U5-OUT_1)
Other:
- board size 215.2 x 179.8 mm -> 131.4 x 111.9 mm
- board text added: "1.65"
- board text added: "3.3V"
- board text added: "5V"
- board text added: "Designed by Adrián Prados López"
- board text added: "MSRL"
- board text added: "Multi Scale Robotics Lab"
- board text added: "PS2"
- board text added: "gnd"
