File: Adrion_1/untitled.kicad_sch (KiCad schematic)
At the start: 1 part, among them U2 STM32G474RET6

Commit message: Modificaciones
Parts:
- removed U2: STM32G474RET6, STM32G474RET6:QFP50P1200X1200X160-64N, symbol STM32G474RET6:STM32G474RET6
- added U2, U5: NUCLEO-G474RE, NUCLEO-G474RE:MODULE_NUCLEO-G474RE, symbol NUCLEO-G474RE_3p:NUCLEO-G474RE
Connections:
- new net EN_GLOBAL: U2.CN10_3 (PB8)
- new net LED_STATUS: U2.CN10_16 (PB12)
- new net PWM_AH: U2.CN10_23 (PA8)
- new net PWM_AL: U2.CN10_21 (PA9)
- new net PWM_BH: U2.CN10_33 (PA10)
- new net PWM_BL: U2.CN10_14 (PA11)

Commit message: Desarrollo
Connections:
- net OVP: now reaches U2.CN10_24 (PB1)
- net LED_STATUS: no longer names the net of U2.CN10_16 (PB12)
Changed lines of the file:
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@@
+	(wire
+		(pts
+			(xy 90.17 111.76) (xy 97.79 111.76)
+		)
+		(stroke
+			(width 0)
+			(type default)
+		)
+	)
 	(wire
 		(pts
@@
 		)
 	)
-	(wire
-		(pts
-			(xy 90.17 101.6) (xy 97.79 101.6)
-		)
-		(stroke
-			(width 0)
-			(type default)
-		)
-	)
 	(hierarchical_label "PWM_AH"
 		(shape output)
@@
 			)
 			(justify right)
-		)
-	)
-	(hierarchical_label "LED_STATUS"
-		(shape output)
-		(at 97.79 101.6 0)
-		(effects
-			(font
-				(size 1.27 1.27)
-			)
-			(justify left)
 		)
 	)
@@
 		)
 	)
+	(hierarchical_label "OVP"
+		(shape input)
+		(at 97.79 111.76 0)
+		(effects
+			(font
+				(size 1.27 1.27)
+			)
+			(justify left)
+		)
+	)

Commit message: Correcciones
Connections:
- net I_Sense: now also U5.CN7_28 (PA0)
- net ENABLE_LDO: now reaches U2.CN10_22 (PB2)
- net NTC_Sense: now reaches U5.CN7_30 (PA1)
Other:
- moved on the sheet: U2B
Changed lines of the file:
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@@
 	(wire
 		(pts
-			(xy 90.17 99.06) (xy 97.79 99.06)
-		)
-		(stroke
-			(width 0)
-			(type default)
-		)
-	)
-	(wire
-		(pts
-			(xy 90.17 111.76) (xy 97.79 111.76)
-		)
-		(stroke
-			(width 0)
-			(type default)
-		)
-	)
-	(wire
-		(pts
-			(xy 35.56 124.46) (xy 44.45 124.46)
-		)
-		(stroke
-			(width 0)
-			(type default)
-		)
-	)
-	(wire
-		(pts
-			(xy 35.56 111.76) (xy 44.45 111.76)
-		)
-		(stroke
-			(width 0)
-			(type default)
-		)
-	)
-	(wire
-		(pts
-			(xy 34.29 86.36) (xy 44.45 86.36)
-		)
-		(stroke
-			(width 0)
-			(type default)
-		)
-	)
-	(wire
-		(pts
-			(xy 35.56 109.22) (xy 44.45 109.22)
+			(xy 91.44 99.06) (xy 99.06 99.06)
+		)
+		(stroke
+			(width 0)
+			(type default)
+		)
+	)
+	(wire
+		(pts
+			(xy 91.44 111.76) (xy 99.06 111.76)
+		)
+		(stroke
+			(width 0)
+			(type default)
+		)
+	)
+	(wire
+		(pts
+			(xy 91.44 58.42) (xy 99.06 58.42)
+		)
+		(stroke
+			(width 0)
+			(type default)
+		)
+	)
+	(wire
+		(pts
+			(xy 36.83 124.46) (xy 45.72 124.46)
+		)
+		(stroke
+			(width 0)
+			(type default)
+		)
+	)
+	(wire
+		(pts
+			(xy 36.83 111.76) (xy 45.72 111.76)
+		)
+		(stroke
+			(width 0)
+			(type default)
+		)
+	)
+	(wire
+		(pts
+			(xy 35.56 86.36) (xy 45.72 86.36)
+		)
+		(stroke
+			(width 0)
+			(type default)
+		)
+	)
+	(wire
+		(pts
+			(xy 36.83 109.22) (xy 45.72 109.22)
+		)
+		(stroke
+			(width 0)
+			(type default)
+		)
+	)
+	(wire
+		(pts
+			(xy 91.44 109.22) (xy 96.52 109.22)
+		)
+		(stroke
+			(width 0)
+			(type default)
+		)
+	)
+	(wire
+		(pts
+			(xy 91.44 60.96) (xy 99.06 60.96)
 		)
 		(stroke
@@
 	(hierarchical_label "PWM_AH"
 		(shape output)
-		(at 35.56 111.76 180)
+		(at 36.83 111.76 180)
 		(effects
 			(font
@@
 	(hierarchical_label "PWM_BH"
 		(shape output)
-		(at 35.56 124.46 180)
+		(at 36.83 124.46 180)
 		(effects
 			(font
@@
 	(hierarchical_label "EN_GLOBAL"
 		(shape output)
-		(at 34.29 86.36 180)
+		(at 35.56 86.36 180)
 		(effects
 			(font
@@
 	(hierarchical_label "OVP"
 		(shape input)
-		(at 97.79 111.76 0)
-		(effects
-			(font
-				(size 1.27 1.27)
-			)
-			(justify left)
-		)
-	)
-	(hierarchical_label "VBUS_SENSE"
+		(at 99.06 111.76 0)
+		(effects
+			(font
+				(size 1.27 1.27)
+			)
+			(justify left)
+		)
+	)
+	(hierarchical_label "ENABLE_LDO"
+		(shape output)
+		(at 96.52 109.22 0)
+		(effects
+			(font
+				(size 1.27 1.27)
+			)
+			(justify left)
+		)
+	)
+	(hierarchical_label "PWM_BL"
+		(shape output)
+		(at 99.06 99.06 0)
+		(effects
+			(font
+				(size 1.27 1.27)
+			)
+			(justify left)
+		)
+	)
+	(hierarchical_label "NTC_Sense"
 		(shape input)
 		(at 99.06 60.96 0)
@@
 		)
 	)
-	(hierarchical_label "PWM_BL"
-		(shape output)
-		(at 97.79 99.06 0)
-		(effects
-			(font
-				(size 1.27 1.27)
-			)
-			(justify left)
-		)
-	)
 	(hierarchical_label "PWM_AL"
 		(shape output)
-		(at 35.56 109.22 180)
+		(at 36.83 109.22 180)
 		(effects
 			(font
@@
 	(symbol
 		(lib_id "NUCLEO-G474RE_3p:NUCLEO-G474RE")
-		(at 67.31 106.68 0)
+		(at 68.58 106.68 0)
 		(unit 2)
 		(exclude_from_sim no)
@@
 		(fields_autoplaced yes)
 		(property "Reference" "U2"
-			(at 67.31 76.2 0)
+			(at 68.58 76.2 0)
 			(effects
 				(font
@@
 		)
 		(property "Value" "NUCLEO-G474RE"
-			(at 67.31 78.74 0)
+			(at 68.58 78.74 0)
 			(effects
 				(font
@@
 		)
 		(property "Footprint" "NUCLEO-G474RE:MODULE_NUCLEO-G474RE"
-			(at 67.31 106.68 0)
+			(at 68.58 106.68 0)
 			(effects
 				(font
@@
 		)
 		(property "Datasheet" ""
-			(at 67.31 106.68 0)
+			(at 68.58 106.68 0)
 			(effects
 				(font
@@
 		)
 		(property "Description" ""
-			(at 67.31 106.68 0)
+			(at 68.58 106.68 0)
 			(effects
 				(font
@@
 		)
 		(property "MF" "STMicroelectronics"
-			(at 67.31 106.68 0)
+			(at 68.58 106.68 0)
 			(effects
 				(font
@@
 		)
 		(property "MAXIMUM_PACKAGE_HEIGHT" "20.7mm"
-			(at 67.31 106.68 0)
+			(at 68.58 106.68 0)
 			(effects
 				(font
@@
 		)
 		(property "Package" "None"
-			(at 67.31 106.68 0)
+			(at 68.58 106.68 0)
 			(effects
 				(font
@@
 		)
 		(property "Price" "None"
-			(at 67.31 106.68 0)
+			(at 68.58 106.68 0)
 			(effects
 				(font
@@
 		)
 		(property "Check_prices" "https://www.snapeda.com/parts/NUCLEO-G474RE/STMicroelectronics/view-part/?ref=eda"
-			(at 67.31 106.68 0)
+			(at 68.58 106.68 0)
 			(effects
 				(font
@@
 		)
 		(property "STANDARD" "Manufacturer Recommendations"
-			(at 67.31 106.68 0)
+			(at 68.58 106.68 0)
 			(effects
 				(font
@@
 		)
 		(property "PARTREV" "17"
-			(at 67.31 106.68 0)
+			(at 68.58 106.68 0)
 			(effects
 				(font
@@
 		)
 		(property "SnapEDA_Link" "https://www.snapeda.com/parts/NUCLEO-G474RE/STMicroelectronics/view-part/?ref=snap"
-			(at 67.31 106.68 0)
+			(at 68.58 106.68 0)
 			(effects
 				(font
@@
 		)
 		(property "MP" "NUCLEO-G474RE"
-			(at 67.31 106.68 0)
+			(at 68.58 106.68 0)
 			(effects
 				(font
@@
 		)
 		(property "Purchase-URL" "https://www.snapeda.com/api/url_track_click_mouser/?unipart_id=3662258&manufacturer=STMicroelectronics&part_name=NUCLEO-G474RE&search_term=None"
-			(at 67.31 106.68 0)
+			(at 68.58 106.68 0)
 			(effects
 				(font
@@
 		)
 		(property "Description_1" "STM32G474 Nucleo-64 STM32G4 ARM® Cortex®-M4 MCU 32-Bit Embedded Evaluation Board"
-			(at 67.31 106.68 0)
+			(at 68.58 106.68 0)
 			(effects
 				(font
@@
 		)
 		(property "Availability" "In Stock"
-			(at 67.31 106.68 0)
+			(at 68.58 106.68 0)
 			(effects
 				(font
@@
 		)
 		(property "MANUFACTURER" "STmicroelectronics"
-			(at 67.31 106.68 0)
-			(effects
-				(font
+			(at 68.58 106.68 0)
+			(effects
+				(font

Commit message: Footprints
Connections:
- net ENABLE_LDO: no longer names the net of U2.CN10_22 (PB2)
- net NTC_Sense: no longer names the net of U5.CN7_30 (PA1)
- net OVP: no longer names the net of U2.CN10_24 (PB1)
Changed lines of the file:
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@@
-	(wire
-		(pts
-			(xy 91.44 111.76) (xy 99.06 111.76)
-		)
-		(stroke
-			(width 0)
-			(type default)
-		)
-	)
 	(wire
 		(pts
@@
 		)
 	)
-	(wire
-		(pts
-			(xy 91.44 109.22) (xy 96.52 109.22)
-		)
-		(stroke
-			(width 0)
-			(type default)
-		)
-	)
-	(wire
-		(pts
-			(xy 91.44 60.96) (xy 99.06 60.96)
-		)
-		(stroke
-			(width 0)
-			(type default)
-		)
-	)
 	(hierarchical_label "PWM_AH"
 		(shape output)
@@
 		)
 	)
-	(hierarchical_label "OVP"
-		(shape input)
-		(at 99.06 111.76 0)
-		(effects
-			(font
-				(size 1.27 1.27)
-			)
-			(justify left)
-		)
-	)
-	(hierarchical_label "ENABLE_LDO"
-		(shape output)
-		(at 96.52 109.22 0)
-		(effects
-			(font
-				(size 1.27 1.27)
-			)
-			(justify left)
-		)
-	)
 	(hierarchical_label "PWM_BL"
 		(shape output)
@@
 		(effects
 			(font
-				(size 1.27 1.27)
-			)
-			(justify left)
-		)
-	)
-	(hierarchical_label "NTC_Sense"
-		(shape input)
-		(at 99.06 60.96 0)
-		(effects
-			(font

Commit message: meduelelacabeza
Parts:
- removed U2, U5: NUCLEO-G474RE, NUCLEO-G474RE:MODULE_NUCLEO-G474RE, symbol NUCLEO-G474RE_3p:NUCLEO-G474RE
- added J6, J7: M20-7821546, M20-7821546:HARWIN_M20-7821546, symbol M20-7821546:M20-7821546
- added U6: NUCLEO-G431KB, NUCLEO-G431KB:MODULE_NUCLEO-G431KB, symbol NUCLEO-G431KB:NUCLEO-G431KB

Commit message: Mamita he empezado el layout. Vaya show
Parts:
- removed U6: NUCLEO-G431KB, NUCLEO-G431KB:MODULE_NUCLEO-G431KB, symbol NUCLEO-G431KB:NUCLEO-G431KB
- added U3: NUCLEO-G431KB, MODULE_NUCLEO-G431KB:MODULE_NUCLEO-G431KB, symbol NUCLEO-G431KB:NUCLEO-G431KB
- J6, J7: footprint M20-7821546:HARWIN_M20-7821546 -> HARWIN_M20-7821546:HARWIN_M20-7821546
Connections:
- net I_Sense: now also J6.11 (PA1(A1))
- net PWM_AH: now also J7.12 (PA8(D9))
- net PWM_AL: now also J6.6 (PA7(A6))
- net PWM_BH: now also J7.1 (PA9(D1))
- net PWM_BL: now also J7.6 (PB0(D3))
- net GND: now reaches J7.4 (GND_CN4)
- net GND: now also J6.2 (GND_CN3)
- net EN_A: now reaches J7.5 (PA12(D2))
- net EN_B: now reaches J7.7 (PB7(D4))
- net 5V: now reaches J6.4 (5V)
- no-connect marks 0 -> 54
Other:
- moved on the sheet: J6, J7

Commit message: FirstPrototype
First Prototype sent
Parts:
- removed J6, J7: M20-7821546, HARWIN_M20-7821546:HARWIN_M20-7821546, symbol M20-7821546:M20-7821546
- removed U3: NUCLEO-G431KB, MODULE_NUCLEO-G431KB:MODULE_NUCLEO-G431KB, symbol NUCLEO-G431KB:NUCLEO-G431KB
- added J8, J9: 6-534237-3, TE_6-534237-3:TE_6-534237-3, symbol 6-534237-3:6-534237-3
Connections:
- net 5V: now also J9.4 (5V)
- net EN_A: now also J8.5 (PA12(D2))
- net EN_B: now also J8.7 (PB7(D4))
- net GND: now also J8.4 (GND), J9.2 (GND)
- net I_Sense: now also J9.11 (PA1(A1))
- net PWM_AH: now also J8.12 (PA8(D9))
- net PWM_AL: now also J9.6 (PA7(A6))
- net PWM_BH: now also J8.1 (PA9(D1))
- net PWM_BL: now also J8.6 (PB0(D3))
- no-connect marks 54 -> 20
